Commit message: Update firefly.xacro

File: quad_control/firefly_link_attached/firefly.xacro (robot description, xacro)
@@ -38,5 +38,5 @@
   <xacro:property name="rotor_drag_coefficient" value="8.06428e-05" />
   <xacro:property name="rolling_moment_coefficient" value="0.000001" />
-  <xacro:property name="link_1_mass" value="0.1" /> <!-- [kg] -->
+  <xacro:property name="link_1_mass" value="0.1" /> <!-- [kg] -->			<!--NEW LINES ADDED FOR THE LINK !!!-->
   <xacro:property name="link_1_width" value="0.025" /> <!-- [m] -->
   <xacro:property name="link_1_height" value="0.25" /> <!-- [m] -->
@@ -45,4 +45,5 @@
     <inertia ixx="0.0347563" ixy="0.0" ixz="0.0" iyy="0.0458929" iyz="0.0" izz="0.0977" /> <!-- [kg m^2] [kg m^2] [kg m^2] [kg m^2] [kg m^2] [kg m^2] -->
   </xacro:property>
+  <!-- NEW LINES ADDED !!! FOR THE LINK INERTIA!! -->
   <xacro:property name="link_1_inertia">
     <inertia ixx="${link_1_mass*(link_1_width*link_1_width + link_1_height*link_1_height)/12}" ixy="0.0" ixz="0.0" iyy="${link_1_mass*(link_1_width*link_1_width + link_1_height*link_1_height)/12}" iyz="0.0" izz="${link_1_mass*(link_1_width*link_1_width + link_1_height*link_1_width)/12}" /> <!-- [kg m^2] [kg m^2] [kg m^2] [kg m^2] [kg m^2] [kg m^2] -->
@@ -66,10 +67,18 @@
     <xacro:insert_block name="body_inertia" />
   </xacro:multirotor_base_macro>
-  <!-- Instantiate manipulator link once -->
+  <!-- NEW LINES ADDED !! Instantiate manipulator link once!!! -->
   <xacro:firefly_manipulator
     robot_namespace="${namespace}"
+    motor_constant="${motor_constant}"
+    moment_constant="${moment_constant}"
+    time_constant_up="${time_constant_up}"
+    time_constant_down="${time_constant_down}"
+    max_rot_velocity="${max_rot_velocity}"
+    motor_number="0"
     mass="${link_1_mass}"
     width="${link_1_width}"
     height="${link_1_height}"
+    direction="cw"
+    color = "Blue"
     >
     <xacro:insert_block name="link_1_inertia" />
