Commit message: Update multirotor_base.xacro

File: quad_control/firefly_link_attached/multirotor_base.xacro (robot description, xacro)
@@ -58,7 +58,7 @@
       </visual>
       <collision>
-        <origin xyz="0 0 ${body_height/4}" rpy="0 0 0" />
+        <origin xyz="0 0 ${body_height/4}" rpy="0 0 0" />	<!--I CHANGED THE BOUNDING BOX OF THE QUAD - IT WAS TOO BIG! -->
         <geometry>
-          <box size="${body_width/2} ${body_width/2} ${body_height/2}" /> <!-- [m] [m] [m] -->
+          <box size="${body_width} ${body_width} ${0.75*body_height}" /> <!-- [m] [m] [m] -->
         </geometry>
       </collision>
